Commit message: Remove .png file calls in urdf

File: tugbot_description/urdf/model.urdf (robot description, URDF)
Before this commit: robot tugbot, 10 links, 9 joints
Links:
- link base_link: geometry visual mesh filename=package://tugbot_description/meshes/base/movai_logo.dae; visual mesh filename=package://tugbot_description/meshes/base/tugbot_simp.dae
